Commit message: 决策更新+点云分割

File: rm_description/urdf/infantry.urdf.xacro (robot description, xacro)
@@ -1,6 +1,12 @@
 <?xml version="1.0" encoding="utf-8"?>
-<robot name="sentry"
-  xmlns:xacro="http://ros.org/wiki/xacro">
-  <link name="base_link"/>
+<robot name="sentry" xmlns:xacro="http://ros.org/wiki/xacro">
+  <xacro:macro name="box_inertia" params="m w h d">
+    <inertial>
+      <mass value="${m}"/>
+      <inertia ixx="${(m/12) * (h*h + d*d)}" ixy="0.0" ixz="0.0"
+               iyy="${(m/12) * (w*w + d*d)}" iyz="0.0"
+               izz="${(m/12) * (w*w + h*h)}"/>
+    </inertial>
+  </xacro:macro>
   <link name="base_footprint"/>
   <joint name="base_footprint_joint" type="fixed">
@@ -9,10 +15,82 @@
     <child link="base_link" />
   </joint>
-  <link name="livox_frame"/>
+  <link name="base_link">
+    <visual>
+      <origin xyz="0 0 0.1" rpy="0 0 0"/>
+      <geometry>
+        <box size="0.4 0.3 0.2"/>
+      </geometry>
+      <material name="blue">
+        <color rgba="0.1 0.1 0.8 1"/>
+      </material>
+    </visual>
+    <collision>
+      <origin xyz="0 0 0.1" rpy="0 0 0"/>
+      <geometry>
+        <box size="0.4 0.3 0.2"/>
+      </geometry>
+    </collision>
+    <xacro:box_inertia m="10.0" w="0.4" h="0.3" d="0.2"/>
+  </link>
+  <link name="livox_frame">
+    <visual>
+      <geometry>
+        <cylinder radius="0.03" length="0.05"/>
+      </geometry>
+      <material name="black">
+        <color rgba="0.1 0.1 0.1 1"/>
+      </material>
+    </visual>
+    <collision>
+      <geometry>
+        <cylinder radius="0.03" length="0.05"/>
+      </geometry>
+    </collision>
+    <xacro:box_inertia m="0.5" w="0.05" h="0.05" d="0.05"/>
+  </link>
   <joint name="lidar_joint" type="fixed">
-    <origin xyz="0 0 0" rpy="0 0 0" />
+    <origin xyz="0 0 0.25" rpy="0 0 0" />
     <parent link="base_link" />
     <child link="livox_frame" />
-    <axis xyz="0 0 0" />
   </joint>
+  <gazebo>
+    <plugin filename="ignition-gazebo-velocity-control-system" name="ignition::gazebo::systems::VelocityControl">
+      <link_name>base_footprint</link_name>
+      <link_name>base_link</link_name>
+      <topic>/cmd_vel</topic>
+    </plugin>
+    <plugin filename="ignition-gazebo-odometry-publisher-system" name="ignition::gazebo::systems::OdometryPublisher">
+      <odom_frame>odom</odom_frame>
+      <robot_base_frame>base_footprint</robot_base_frame>
+      <odom_topic>/odom</odom_topic>
+      <tf_topic>/tf</tf_topic>
+      <dimensions>2</dimensions>
+      <odom_publish_frequency>50</odom_publish_frequency>
+    </plugin>
+  </gazebo>
+  <gazebo reference="livox_frame">
+    <sensor name="lidar" type="gpu_lidar">
+      <ignition_frame_id>livox_frame</ignition_frame_id>
+      <pose>0 0 0 0 0 0</pose>
+      <topic>/scan</topic>
+      <update_rate>10</update_rate>
+      <ray>
+        <scan>
+          <horizontal>
+            <samples>360</samples>
+            <resolution>1</resolution>
+            <min_angle>-3.14159</min_angle>
+            <max_angle>3.14159</max_angle>
+          </horizontal>
+        </scan>
+        <range>
+          <min>0.15</min>
+          <max>12.0</max>
+          <resolution>0.01</resolution>
+        </range>
+      </ray>
+      <always_on>1</always_on>
+      <visualize>true</visualize>
+    </sensor>
+  </gazebo>
 </robot>
